File: olice/test1.kicad_pcb (KiCad board)
At the start: 2 copper layers, 249.9 x 88.1 mm, 108 parts, among them J1 AVR-ISP-6, K1 KEYSW, K10 KEYSW, K11 KEYSW, K12 KEYSW, K13 KEYSW, K14 KEYSW, K15 KEYSW, K16 KEYSW, K17 KEYSW, K18 KEYSW, K19 KEYSW, K2 KEYSW, K20 KEYSW, K21 KEYSW, K22 KEYSW, K23 KEYSW, K24 KEYSW, K25 KEYSW, K26 KEYSW, K27 KEYSW, K28 KEYSW, K29 KEYSW, K3 KEYSW, K30 KEYSW, K31 KEYSW, K32 KEYSW, K33 KEYSW, K34 KEYSW, K35 KEYSW, K36 KEYSW, K37 KEYSW, K38 KEYSW, K39 KEYSW, K4 KEYSW, K40 KEYSW, K41 KEYSW, K42 KEYSW, K43 KEYSW, K44 KEYSW, K5 KEYSW, K6 KEYSW, K7 KEYSW, K8 KEYSW, K9 KEYSW, SW1 SW_PUSH, U1 ATmega32U4-AU, Y1 XTAL

Commit message: recreated updated gerbers with added keys on bottom row, recreated plate file with correct switch hole dimensions
Parts:
- added D46: D, Diode_SMD:D_SOD-123, B.Cu at (61.7, 98.3)
- added D47: D, Diode_SMD:D_SOD-123, B.Cu at (218.7, 100.3)
- added K45: KEYSW, Button_Switch_Keyboard:SW_Cherry_MX_1.00u_Plate, F.Cu at (72.4, 94.5)
- added K46: KEYSW, Button_Switch_Keyboard:SW_Cherry_MX_1.00u_Plate, F.Cu at (228.0, 93.8)
Routing:
- net col9: track 136.1 -> 142.7 mm, vias 1 -> 0
- net Net-(D47-Pad2): track 0.00 -> 4.32 mm
- net Net-(D46-Pad2): track 0.00 -> 4.04 mm
- net col2: track 150.3 -> 152.5 mm
- net row3: track 254.0 -> 252.6 mm
- net col10: track 165.5 -> 164.8 mm
- net col11: track 191.3 -> 190.6 mm
