File: olice/test1.sch (KiCad schematic (older format))
At the start: 108 parts, among them J1 AVR-ISP-6, K1 KEYSW, K10 KEYSW, K11 KEYSW, K12 KEYSW, K13 KEYSW, K14 KEYSW, K15 KEYSW, K16 KEYSW, K17 KEYSW, K18 KEYSW, K19 KEYSW, K2 KEYSW, K20 KEYSW, K21 KEYSW, K22 KEYSW, K23 KEYSW, K24 KEYSW, K25 KEYSW, K26 KEYSW, K27 KEYSW, K28 KEYSW, K29 KEYSW, K3 KEYSW, K30 KEYSW, K31 KEYSW, K32 KEYSW, K33 KEYSW, K34 KEYSW, K35 KEYSW, K36 KEYSW, K37 KEYSW, K38 KEYSW, K39 KEYSW, K4 KEYSW, K40 KEYSW, K41 KEYSW, K42 KEYSW, K43 KEYSW, K44 KEYSW, K5 KEYSW, K6 KEYSW, K7 KEYSW, K8 KEYSW, K9 KEYSW, SW1 SW_PUSH, U1 ATmega32U4-AU, Y1 XTAL

Commit message: recreated updated gerbers with added keys on bottom row, recreated plate file with correct switch hole dimensions
Parts:
- added D46, D47: D, Diode_SMD:D_SOD-123, symbol Device:D
- added K45, K46: KEYSW, Button_Switch_Keyboard:SW_Cherry_MX_1.00u_Plate, symbol keyboard_parts:KEYSW
Connections:
- net col2: now also K45.1
- net col9: now also K46.1
- net row3: now also D46.1 (K), D47.1 (K)
- new net: D46.2 (A), K45.2
- new net: D47.2 (A), K46.2
Changed lines of the file:
@@
 Connection ~ 6350 4050
 Wire Wire Line
-	7550 3850 10100 3850
+	7550 3850 9250 3850
 Wire Wire Line
-	14350 3850 16900 3850
+	14350 3850 15200 3850
 NoConn ~ 1550 3150
 NoConn ~ 7150 2750
@@
 Text GLabel 2250 3050 2    50   Input ~ 0
 col2
+$Comp
+L Device:D D46
+U 1 1 607FBDCA
+P 9250 3700
+F 0 "D46" V 9296 3620 50  0000 R CNN
+F 1 "D" V 9205 3620 50  0000 R CNN
+F 2 "Diode_SMD:D_SOD-123" H 9250 3700 50  0001 C CNN
+F 3 "~" H 9250 3700 50  0001 C CNN
+	1    9250 3700
+	0    -1   -1   0
+$EndComp
+Connection ~ 9250 3850
+Wire Wire Line
+	9250 3850 10100 3850
+$Comp
+L keyboard_parts:KEYSW K45
+U 1 1 607FC407
+P 9550 3550
+F 0 "K45" H 9550 3783 60  0000 C CNN
+F 1 "KEYSW" H 9550 3450 60  0001 C CNN
+F 2 "Button_Switch_Keyboard:SW_Cherry_MX_1.00u_Plate" H 9550 3550 60  0001 C CNN
+F 3 "" H 9550 3550 60  0000 C CNN
+	1    9550 3550
+	1    0    0    -1
+$EndComp
+Wire Wire Line
+	9850 3050 9850 3550
+Connection ~ 9850 3050
+$Comp
+L Device:D D47
+U 1 1 608063E0
+P 15200 3700
+F 0 "D47" V 15246 3620 50  0000 R CNN
+F 1 "D" V 15155 3620 50  0000 R CNN
+F 2 "Diode_SMD:D_SOD-123" H 15200 3700 50  0001 C CNN
+F 3 "~" H 15200 3700 50  0001 C CNN
+	1    15200 3700
+	0    -1   -1   0
+$EndComp
+Connection ~ 15200 3850
+Wire Wire Line
+	15200 3850 16900 3850
+$Comp
+L keyboard_parts:KEYSW K46
+U 1 1 6080699D
+P 15500 3550
+F 0 "K46" H 15500 3783 60  0000 C CNN
+F 1 "KEYSW" H 15500 3450 60  0001 C CNN
+F 2 "Button_Switch_Keyboard:SW_Cherry_MX_1.00u_Plate" H 15500 3550 60  0001 C CNN
+F 3 "" H 15500 3550 60  0000 C CNN
+	1    15500 3550
+	1    0    0    -1
+$EndComp
+Wire Wire Line
+	15800 3050 15800 3550
+Connection ~ 15800 3050
 $EndSCHEMATC
